File: Kicad/Interface_CM108.kicad_sch (KiCad schematic)
At the start: 38 parts, among them IC1 CM108B, J1 USB_C_Receptacle_USB2.0_16P, J2 RJ45, Q1 BC546ABU, T1 Transformer_1P_1S, T2 Transformer_1P_1S, U1 93C46, U2 PC318

Commit message: Revision v4
Parts:
- removed 3.3V1: 3.3V, TestPoint:TestPoint_Pad_D1.0mm, symbol Connector:TestPoint_Flag
- added C13: 100nF, Capacitor_THT:C_Disc_D3.8mm_W2.6mm_P2.50mm, symbol Device:C_Small
- added C14: 10µ, Capacitor_THT:CP_Radial_D5.0mm_P2.00mm, symbol Device:C_Polarized
- added C15: 10µF, Capacitor_THT:C_Disc_D3.8mm_W2.6mm_P2.50mm, symbol Device:C_Small
- added L4, L5: Ferrite_Bead, Inductor_SMD:L_1210_3225Metric, symbol cm108b-eval-rescue:L_Core_Ferrite-Device
- C10: value 470μ -> 100μF; footprint Capacitor_THT:CP_Radial_D10.0mm_P5.00mm -> Capacitor_THT:CP_Radial_D5.0mm_P2.00mm
- C11: value 1µ -> 1µF; footprint Capacitor_THT:CP_Radial_D4.0mm_P1.50mm -> Capacitor_THT:CP_Radial_D5.0mm_P2.00mm
- C12: value 4.7µ -> 1µF; footprint Capacitor_THT:CP_Radial_D4.0mm_P1.50mm -> Capacitor_THT:CP_Radial_D5.0mm_P2.00mm
- C3: value 4.7µ -> 10µ; footprint Capacitor_THT:CP_Radial_D4.0mm_P1.50mm -> Capacitor_THT:CP_Radial_D5.0mm_P2.00mm
- C5: value 4.7µ -> 10µ; footprint Capacitor_THT:CP_Radial_D4.0mm_P1.50mm -> Capacitor_THT:CP_Radial_D5.0mm_P2.00mm; KiLib_Generator (none) -> capacitor/THT/other
- R4, R5: value 22 -> 39
- R7: value 1.5k -> 8.2k; KiLib_Generator (none) -> resistor/THT
Connections:
- net MIC_IN: now also R7.1; no longer C11.1
- net USB+: no longer R7.2
- net VBUS: now also J1.A4 (VBUS), J1.A9 (VBUS), J1.B4 (VBUS), J1.B9 (VBUS), L1.1, L4.1; no longer C1.1, C2.1, C3.1, C4.1, C5.1, C6.1, IC1.29 (AVDD1), IC1.34 (AVDD2), IC1.35 (DVDD), IC1.38 (MSEL), L1.2, R2.1, U1.8 (VCC)
- net at IC1.37 (AREG36): now also C14.1
- net at IC1.8 (DREG18): now also C13.2
- net +3.3V renamed +3V3
- net +3V3: now also IC1.38 (MSEL); no longer R7.1
- net GND renamed GNDD
- net GNDD: now also C13.1, C15.1, L5.1; no longer C3.2, C4.2, C6.2, C9.2, IC1.24 (AVSS1), IC1.33 (AVSS2), T1.3 (AB), T2.1 (AA)
- new net: C11.1, R7.2
- new net +5VA: C3.1, C4.1, C6.1, IC1.29 (AVDD1), IC1.34 (AVDD2), L1.2
- new net +5VD: C1.1, C2.1, C5.1, IC1.35 (DVDD), L4.2, R2.1, U1.8 (VCC)
- new net GNDA: C14.2, C15.2, C3.2, C4.2, C6.2, C9.2, IC1.24 (AVSS1), IC1.33 (AVSS2), L5.2, T1.3 (AB), T2.1 (AA)
- no-connect marks 23 -> 21
Other:
- note added: "Changelog v4 - Enlevé pull-up non nécessaire sur D+. - Correction câblage MSEL - Ajout condo sur DREG18, AREG36 - Condo DREG33 C12 1µF => 100 nF - Modification MIC_IN path - C10 path audio in 470 µF => 100µF - Modification ferrites + condos sur VBUS - Séparation GNDA/GNDD"
- moved on the sheet: 5V1, C1, C10, C11, C12, C2, C3, C4, C6, C9, D1, IC1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

Commit message: Add files via upload
Parts:
- R4, R5: value 39 -> 22
Changed lines of the file:
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@@
 			)
 		)
-		(property "Value" "39"
+		(property "Value" "22"
 			(at 73.66 36.4744 90)
 			(show_name no)
@@
 			)
 		)
-		(property "Value" "39"
+		(property "Value" "22"
 			(at 73.66 47.0916 90)
 			(show_name no)
